File: N-P-MOSFET_adapter/N-P-MOSFET_adapter.brd (EAGLE design)
At the start: 13 x 8.2 mm, 13 parts, among them Q1 BSS83P, Q2 BSS83P, Q3 BSS138, Q4 BSS138

Commit message: schematic
Parts:
- removed JP6: (no value), my-pinhead:1X01_BARE
- added JP1: (no value), my-pinhead:1X01_BARE
- Q2: value BSS83P -> BSS138
- Q3: value BSS138 -> BSS83P
- moved Q2 9.21 mm to (11.1, 5.65), flipped to the bottom
- moved Q3 9.21 mm to (1.91, 5.65), flipped to the top
- moved JP4 2.54 mm to (3.97, 1.43)
- moved JP5 2.54 mm to (1.43, 1.43)
- moved R2 2.29 mm to (7.52, 5.71), flipped to the bottom, turned to 90 degrees
- moved R3 2.29 mm to (5.24, 5.71), flipped to the top, turned to 270 degrees
Connections:
- net D1: now also JP5.1, Q3.3; no longer JP6.1, Q2.3
- net D2: now also Q2.3; no longer Q3.3
- net G1: now also JP4.1, Q3.1, R3.1; no longer JP5.1, Q2.1, R2.1
- net G2: now also Q2.1, R2.2; no longer Q3.1, R3.2
- net PWR: now also JP1.1, R2.1, R3.2; no longer JP4.1, R2.2, R3.1
Changed lines of the file:
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@@
 <elements>
 <element name="Q1" library="my-mosfet" package="SOT23" value="BSS83P" x="11.1125" y="5.6515" rot="R180"/>
-<element name="Q2" library="my-mosfet" package="SOT23" value="BSS83P" x="1.905" y="5.6515" rot="R180"/>
+<element name="Q3" library="my-mosfet" package="SOT23" value="BSS83P" x="1.905" y="5.6515" rot="R180"/>
 <element name="R1" library="rcl" library_urn="urn:adsk.eagle:library:334" package="R0805" package3d_urn="urn:adsk.eagle:package:23553/2" value="" x="7.52475" y="5.715" rot="R270"/>
-<element name="R2" library="rcl" library_urn="urn:adsk.eagle:library:334" package="R0805" package3d_urn="urn:adsk.eagle:package:23553/2" value="" x="5.23875" y="5.715" rot="R270"/>
+<element name="R3" library="rcl" library_urn="urn:adsk.eagle:library:334" package="R0805" package3d_urn="urn:adsk.eagle:package:23553/2" value="" x="5.23875" y="5.715" rot="R270"/>
 <element name="JP2" library="my-pinhead" package="1X01_BARE" value="" x="11.58875" y="1.42875" rot="MR0"/>
 <element name="JP3" library="my-pinhead" package="1X01_BARE" value="" x="9.04875" y="1.42875" rot="MR0"/>
-<element name="JP4" library="my-pinhead" package="1X01_BARE" value="" x="6.50875" y="1.42875" rot="MR0"/>
-<element name="JP5" library="my-pinhead" package="1X01_BARE" value="" x="3.96875" y="1.42875" rot="MR0"/>
-<element name="JP6" library="my-pinhead" package="1X01_BARE" value="" x="1.42875" y="1.42875" rot="MR0"/>
-<element name="Q3" library="my-mosfet" package="SOT23" value="BSS138" x="11.1125" y="5.6515" rot="MR180"/>
+<element name="JP1" library="my-pinhead" package="1X01_BARE" value="" x="6.50875" y="1.42875" rot="MR0"/>
+<element name="JP4" library="my-pinhead" package="1X01_BARE" value="" x="3.96875" y="1.42875" rot="MR0"/>
+<element name="JP5" library="my-pinhead" package="1X01_BARE" value="" x="1.42875" y="1.42875" rot="MR0"/>
+<element name="Q2" library="my-mosfet" package="SOT23" value="BSS138" x="11.1125" y="5.6515" rot="MR180"/>
 <element name="Q4" library="my-mosfet" package="SOT23" value="BSS138" x="1.905" y="5.6515" rot="MR180"/>
-<element name="R3" library="rcl" library_urn="urn:adsk.eagle:library:334" package="R0805" package3d_urn="urn:adsk.eagle:package:23553/2" value="" x="7.52475" y="5.715" rot="MR90"/>
+<element name="R2" library="rcl" library_urn="urn:adsk.eagle:library:334" package="R0805" package3d_urn="urn:adsk.eagle:package:23553/2" value="" x="7.52475" y="5.715" rot="MR90"/>
 <element name="R4" library="rcl" library_urn="urn:adsk.eagle:library:334" package="R0805" package3d_urn="urn:adsk.eagle:package:23553/2" value="" x="5.23875" y="5.715" rot="MR90"/>
 </elements>
 <signals>
 <signal name="PWR">
-<contactref element="Q2" pad="2"/>
+<contactref element="Q3" pad="2"/>
 <contactref element="Q1" pad="2"/>
 <contactref element="R1" pad="2"/>
-<contactref element="R2" pad="2"/>
+<contactref element="R3" pad="2"/>
 <polygon width="0.3048" layer="1">
 <vertex x="0" y="8.41375"/>
@@
 <vertex x="13.0175" y="8.5725"/>
 </polygon>
-<contactref element="JP4" pad="1"/>
+<contactref element="JP1" pad="1"/>
 <contactref element="R4" pad="1"/>
 <contactref element="Q4" pad="2"/>
-<contactref element="R3" pad="1"/>
-<contactref element="Q3" pad="2"/>
+<contactref element="R2" pad="1"/>
+<contactref element="Q2" pad="2"/>
 <polygon width="0.3048" layer="16">
 <vertex x="0" y="8.255"/>
@@
 <wire x1="11.1125" y1="4.6515" x2="10.19175" y2="4.6355" width="0.3048" layer="1"/>
 <wire x1="10.19175" y1="4.6355" x2="9.04875" y2="3.4925" width="0.3048" layer="1"/>
-<contactref element="Q3" pad="3"/>
+<contactref element="Q2" pad="3"/>
 <wire x1="9.04875" y1="3.4925" x2="9.04875" y2="1.42875" width="0.3048" layer="16"/>
 <wire x1="11.1125" y1="4.6515" x2="10.19175" y2="4.6355" width="0.3048" layer="16"/>
@@
 <contactref element="Q4" pad="1"/>
 <contactref element="R4" pad="2"/>
-<contactref element="Q2" pad="1"/>
-<contactref element="R2" pad="1"/>
-<contactref element="JP5" pad="1"/>
+<contactref element="Q3" pad="1"/>
+<contactref element="R3" pad="1"/>
+<contactref element="JP4" pad="1"/>
 <wire x1="3.96875" y1="6.6675" x2="5.23625" y2="6.6675" width="0.3048" layer="1"/>
 <wire x1="5.23625" y1="6.6675" x2="5.23875" y2="6.665" width="0.3048" layer="1"/>
@@
 </signal>
 <signal name="G2">
-<contactref element="R3" pad="2"/>
-<contactref element="Q3" pad="1"/>
+<contactref element="R2" pad="2"/>
+<contactref element="Q2" pad="1"/>
 <contactref element="Q1" pad="1"/>
 <contactref element="R1" pad="1"/>
@@
 <signal name="D1">
 <contactref element="Q4" pad="3"/>
-<contactref element="Q2" pad="3"/>
-<contactref element="JP6" pad="1"/>
+<contactref element="Q3" pad="3"/>
+<contactref element="JP5" pad="1"/>
 <wire x1="1.42875" y1="3.01625" x2="1.905" y2="3.4925" width="0.3048" layer="1"/>
 <wire x1="1.905" y1="3.4925" x2="1.905" y2="4.6515" width="0.3048" layer="1"/>

Commit message: new adapters
Parts:
- removed R3: (no value), rcl:R0805
- added R5: (no value), rcl:R0805
- moved JP2 10.2 mm to (1.43, 1.43)
- moved JP5 10.2 mm to (11.6, 1.43)
- moved Q3 8.89 mm to (10.8, 5.56)
- moved Q4 8.89 mm to (10.8, 5.56)
- moved R1 6.10 mm to (1.43, 5.56)
- moved Q1 4.13 mm to (6.99, 5.56)
- moved Q2 4.13 mm to (6.99, 5.56)
- moved R2 3.88 mm to (3.65, 5.56), flipped to the top
- moved R4 3.81 mm to (1.43, 5.56), turned to 270 degrees
Connections:
- new net N$3: Q1.1, Q2.1, R1.1
- new net N$4: Q3.1, Q4.1, R4.1
- net D1: now also JP3.1, Q1.3, Q2.3; no longer JP5.1, Q3.3, Q4.3
- net D2: now also JP5.1, Q3.3, Q4.3; no longer JP3.1, Q1.3, Q2.3
- net G1: now also JP2.1, R1.2, R2.1; no longer JP4.1, Q3.1, Q4.1, R3.1, R4.2
- net G2: now also JP4.1, R4.2, R5.1; no longer JP2.1, Q1.1, Q2.1, R1.1, R2.2
- net PWR: now also R2.2, R5.2; no longer R1.2, R2.1, R3.2, R4.1
Routing:
- net N$4: track 0.00 -> 18.4 mm, vias 0 -> 1
- net G2: track 20.6 -> 5.53 mm
- net G1: track 17.9 -> 5.40 mm
- net N$3: track 0.00 -> 12.5 mm, vias 0 -> 1
- net D2: track 9.20 -> 6.91 mm
- net D1: track 6.84 -> 7.96 mm
- added copper zone on layer 1, net N$5
- added copper zone on layer 16, net N$5
Other:
- board size 13 x 8.2 mm -> 13 x 7.9 mm
